File: PCB/Root41-2020/001.brd (EAGLE design)
At the start: 97 x 33.1 mm, 46 parts, among them P1 S6B-ZR-SM4A-TF, T1 NJL7502L, T10 NJL7502L, T11 NJL7502L, T12 NJL7502L, T2 NJL7502L, T3 NJL7502L, T4 NJL7502L, T5 NJL7502L, T6 NJL7502L, T7 NJL7502L, T8 NJL7502L, T9 NJL7502L, U1 STMICROELECTRONICS_STM32L010F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

Commit message: no message
Parts:
- removed C1, C2: 0.1μF, rcl:C0603
- removed R1, R2, R3, R4: 47k, rcl:R0805
- removed U1: STMICROELECTRONICS_STM32L010F4P6STMICROELECTRONICS_STM32L01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, STMicroelectronics - STM32L010F4P6:STMICROELECTRONICS_STM32L010F4P6_3
- P1: value S6B-ZR-SM4A-TF -> (none); device zh:ZH-SM4-SIDE06 -> zh:ZH-SM4-SIDE09
- moved R14 13.0 mm to (4.00, -12.3)
- moved R9 10.8 mm to (16.0, -7.00), flipped to the top, turned to 0 degrees
- moved R13 6.91 mm to (-13.0, -23.1)
- moved R8 5.52 mm to (-10.5, -4.50), flipped to the top, turned to 270 degrees
- moved R15 4.53 mm to (13.0, -23.1)
- moved P1 2.31 mm to (-8.80, -21.0)
- moved U$1 1.02 mm to (0.00, -6.00)
- moved T3 0.30 mm to (-16.0, -4.50)
- moved R12 0.30 mm to (-24.7, -29.0)
- moved R16 0.30 mm to (24.7, -29.0)
Connections:
- removed net N$12: R2.1, U1.1
- removed net NRST: C2.2, R1.2, U1.4
- removed net SCL: P1.4, R3.2, U1.17
- removed net SDA: P1.2, R4.2, U1.18
- net +3V3: no longer C1.2, R1.1, R3.1, R4.1, U1.16, U1.5
- net +5V: now also P1.8; no longer P1.5
- net GND: now also P1.6; no longer C1.1, C2.1, P1.3, R2.2, U1.15
- net MUX: now also P1.7; no longer U1.7
- net NEOPIXEL-SIGNAL: now also P1.9; no longer P1.6
- net S0: now also P1.2; no longer U1.10
- net S1: now also P1.3; no longer U1.11
- net S2: now also P1.4; no longer U1.12
- net S3: now also P1.5; no longer U1.13
Routing:
- net GND: track 0.00 -> 218.9 mm, vias 0 -> 1
- net +3V3: track 0.00 -> 198.1 mm, vias 0 -> 4
- net +5V: track 0.00 -> 188.8 mm, vias 0 -> 4
- net IN6: track 0.00 -> 64.9 mm, vias 0 -> 1
- net N$8: track 0.00 -> 62.4 mm, vias 0 -> 2
- net IN7: track 0.00 -> 58.7 mm, vias 0 -> 1
- net NEOPIXEL-SIGNAL: track 0.00 -> 57.1 mm, vias 0 -> 5
- net MUX: track 0.00 -> 56.9 mm, vias 0 -> 4
- net IN5: track 0.00 -> 42.8 mm
- net IN11: track 0.00 -> 38.6 mm
- net IN0: track 0.00 -> 37.0 mm
- net IN8: track 0.00 -> 36.0 mm, vias 0 -> 2
- net N$9: track 0.00 -> 35.5 mm
- net IN4: track 0.00 -> 31.3 mm
- net N$4: track 0.00 -> 28.9 mm, vias 0 -> 2
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- added copper zone on layer 1, net GND
- added copper zone on layer 16, net GND

Commit message: no message
Parts:
- added U$2: (no value), oshw:OSHW_5MM
Other:
- board text removed: "memo Y:-63mm"

Commit message: 基板設計完了
Parts:
- added R1: 180, rcl:R2012
- added R3: 120k, rcl:R0805
- added TP1, TP3: TPSQTP11R, testpad:TP11R
- added TP2, TP4: TPSQTP11SQ, testpad:TP11SQ
Connections:
- new net N$12: R1.1, TP2.TP
- net +3V3: now also R3.1
- net +5V: now also R1.2
- net GND: now also TP1.TP, TP3.TP
- net IN13: now also R3.2, TP4.TP
Routing:
- net N$4: track 28.9 -> 101.0 mm, vias 2 -> 0
- net IN13: track 0.00 -> 40.3 mm, vias 0 -> 2
- net MUX: track 56.9 -> 18.8 mm, vias 4 -> 2
- net +5V: track 188.8 -> 217.4 mm, vias 4 -> 8
- net IN11: track 38.6 -> 60.4 mm, vias 0 -> 5
- net +3V3: track 198.1 -> 183.2 mm, vias 4 -> 6
- net NEOPIXEL-SIGNAL: track 57.1 -> 42.2 mm, vias 5 -> 1
- net IN6: track 64.9 -> 55.6 mm, vias 1 -> 0
- net S1: track 14.5 -> 21.4 mm, vias 2 -> 0
- net IN4: track 31.3 -> 25.9 mm, vias 0 -> 1
- net IN3: track 15.5 -> 20.8 mm, vias 0 -> 2
- net N$8: track 62.4 -> 57.8 mm
- net IN1: track 26.0 -> 30.4 mm, vias 0 -> 2
- net S0: track 20.9 -> 24.7 mm, vias 0 -> 2
- net N$12: track 0.00 -> 3.26 mm
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Other:
- board text added: "JLCJLCJLCJLC"
