File: PCB/Root41-2020/001.sch (EAGLE design)
At the start: 46 parts, among them P1 S6B-ZR-SM4A-TF, T1 NJL7502L, T10 NJL7502L, T11 NJL7502L, T12 NJL7502L, T2 NJL7502L, T3 NJL7502L, T4 NJL7502L, T5 NJL7502L, T6 NJL7502L, T7 NJL7502L, T8 NJL7502L, T9 NJL7502L, U1 STMICROELECTRONICS_STM32L010F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

Commit message: no message
Parts:
- removed C1, C2: 0.1μF, rcl:C-EUC0603
- removed R1, R2, R3, R4: 47k, rcl:R-EU_R0805
- removed U1: STMICROELECTRONICS_STM32L010F4P6STMICROELECTRONICS_STM32L01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, STMicroelectronics - STM32L010F4P6:STMICROELECTRONICS_STM32L010F4P6STMICROELECTRONICS_STM32L010F4P6_0_3
- P1: value S6B-ZR-SM4A-TF -> (none); device zh:S6B-ZR-SM4A-TF -> zh:S9B-ZR-SM4A-TF
Connections:
- removed net N$12: R2.1, U1.PB9-BOOT0
- removed net NRST: C2.2, R1.2, U1.!RST!
- removed net SCL: P1.4, R3.2, U1.PA9
- removed net SDA: P1.2, R4.2, U1.PA10
- net +3V3: no longer C1.2, R1.1, R3.1, R4.1, U1.VDD, U1.VDDA
- net +5V: now also P1.8; no longer P1.5
- net GND: now also P1.6; no longer C1.1, C2.1, P1.3, R2.2, U1.VSS
- net MUX: now also P1.7; no longer U1.PA1
- net NEOPIXEL-SIGNAL: now also P1.9; no longer P1.6
- net S0: now also P1.2; no longer U1.PA4
- net S1: now also P1.3; no longer U1.PA5
- net S2: now also P1.4; no longer U1.PA6
- net S3: now also P1.5; no longer U1.PA7

Commit message: 基板設計完了
Parts:
- added R1: 180, rcl:R-EU_R2012
- added R3: 120k, rcl:R-EU_R0805
- added TP1, TP3: TPSQTP11R, testpad:TPSQTP11R
- added TP2, TP4: TPSQTP11SQ, testpad:TPSQTP11SQ
Connections:
- new net N$12: R1.1, TP2.TP
- net +3V3: now also R3.1
- net +5V: now also R1.2
- net GND: now also TP1.TP, TP3.TP
- net IN13: now also R3.2, TP4.TP
Changed lines of the file:
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@@
 <part name="+3V7" library="supply1" library_urn="urn:adsk.eagle:library:371" deviceset="+3V3" device=""/>
 <part name="P1" library="zh" deviceset="S9B-ZR-SM4A-TF" device=""/>
+<part name="TP1" library="testpad" library_urn="urn:adsk.eagle:library:385" deviceset="TPSQ" device="TP11R" package3d_urn="urn:adsk.eagle:package:27961/1"/>
+<part name="TP2" library="testpad" library_urn="urn:adsk.eagle:library:385" deviceset="TPSQ" device="TP11SQ" package3d_urn="urn:adsk.eagle:package:27965/1"/>
+<part name="R1" library="rcl" library_urn="urn:adsk.eagle:library:334" deviceset="R-EU_" device="R2012" package3d_urn="urn:adsk.eagle:package:23543/2" value="180"/>
+<part name="GND15" library="supply1" library_urn="urn:adsk.eagle:library:371" deviceset="GND" device=""/>
+<part name="P+15" library="supply1" library_urn="urn:adsk.eagle:library:371" deviceset="+5V" device=""/>
+<part name="TP3" library="testpad" library_urn="urn:adsk.eagle:library:385" deviceset="TPSQ" device="TP11R" package3d_urn="urn:adsk.eagle:package:27961/1"/>
+<part name="TP4" library="testpad" library_urn="urn:adsk.eagle:library:385" deviceset="TPSQ" device="TP11SQ" package3d_urn="urn:adsk.eagle:package:27965/1"/>
+<part name="GND16" library="supply1" library_urn="urn:adsk.eagle:library:371" deviceset="GND" device=""/>
+<part name="R3" library="rcl" library_urn="urn:adsk.eagle:library:334" deviceset="R-EU_" device="R0805" package3d_urn="urn:adsk.eagle:package:23553/2" value="120k"/>
+<part name="+3V2" library="supply1" library_urn="urn:adsk.eagle:library:371" deviceset="+3V3" device=""/>
 </parts>
 <sheets>
@@
 <attribute name="VALUE" x="54.61" y="55.88" size="1.778" layer="96"/>
 </instance>
+<instance part="TP1" gate="G$1" x="20.32" y="27.94" smashed="yes" rot="R270">
+<attribute name="NAME" x="12.7" y="27.94" size="1.778" layer="95"/>
+<attribute name="TP_SIGNAL_NAME" x="19.05" y="25.4" size="1.778" layer="97" rot="R270"/>
+</instance>
+<instance part="TP2" gate="G$1" x="20.32" y="30.48" smashed="yes" rot="R270">
+<attribute name="NAME" x="12.7" y="30.48" size="1.778" layer="95"/>
+<attribute name="TP_SIGNAL_NAME" x="19.05" y="27.94" size="1.778" layer="97" rot="R270"/>
+</instance>
+<instance part="R1" gate="G$1" x="35.56" y="30.48" smashed="yes">
+<attribute name="NAME" x="31.75" y="31.9786" size="1.778" layer="95"/>
+<attribute name="VALUE" x="36.83" y="32.258" size="1.778" layer="96"/>
+</instance>
+<instance part="GND15" gate="1" x="33.02" y="22.86" smashed="yes">
+<attribute name="VALUE" x="30.48" y="20.32" size="1.778" layer="96"/>
+</instance>
+<instance part="P+15" gate="1" x="48.26" y="38.1" smashed="yes">
+<attribute name="VALUE" x="50.8" y="35.56" size="1.778" layer="96"/>
+</instance>
+<instance part="TP3" gate="G$1" x="60.96" y="27.94" smashed="yes" rot="R270">
+<attribute name="NAME" x="53.34" y="27.94" size="1.778" layer="95"/>
+<attribute name="TP_SIGNAL_NAME" x="59.69" y="25.4" size="1.778" layer="97" rot="R270"/>
+</instance>
+<instance part="TP4" gate="G$1" x="60.96" y="30.48" smashed="yes" rot="R270">
+<attribute name="NAME" x="53.34" y="30.48" size="1.778" layer="95"/>
+<attribute name="TP_SIGNAL_NAME" x="59.69" y="27.94" size="1.778" layer="97" rot="R270"/>
+</instance>
+<instance part="GND16" gate="1" x="73.66" y="22.86" smashed="yes">
+<attribute name="VALUE" x="71.12" y="20.32" size="1.778" layer="96"/>
+</instance>
+<instance part="R3" gate="G$1" x="73.66" y="40.64" smashed="yes" rot="R270">
+<attribute name="NAME" x="76.2" y="40.64" size="1.778" layer="95"/>
+<attribute name="VALUE" x="76.2" y="38.1" size="1.778" layer="96"/>
+</instance>
+<instance part="+3V2" gate="G$1" x="73.66" y="50.8" smashed="yes">
+<attribute name="VALUE" x="76.2" y="50.8" size="1.778" layer="96"/>
+</instance>
 </instances>
 <busses>
@@
 <pinref part="U$1" gate="G$1" pin="CHAN13"/>
 <label x="15.24" y="119.38" size="1.778" layer="95"/>
+</segment>
+<segment>
+<wire x1="73.66" y1="30.48" x2="73.66" y2="33.02" width="0.1524" layer="91"/>
+<wire x1="73.66" y1="33.02" x2="78.74" y2="33.02" width="0.1524" layer="91"/>
+<label x="81.28" y="33.02" size="1.778" layer="95"/>
+<wire x1="73.66" y1="33.02" x2="73.66" y2="35.56" width="0.1524" layer="91"/>
+<junction x="73.66" y="33.02"/>
+<pinref part="R3" gate="G$1" pin="2"/>
+<pinref part="TP4" gate="G$1" pin="TP"/>
+<wire x1="63.5" y1="30.48" x2="73.66" y2="30.48" width="0.1524" layer="91"/>
 </segment>
 </net>
@@
 <pinref part="P1" gate="G$1" pin="6"/>
 </segment>
+<segment>
+<pinref part="TP1" gate="G$1" pin="TP"/>
+<wire x1="22.86" y1="27.94" x2="33.02" y2="27.94" width="0.1524" layer="91"/>
+<wire x1="33.02" y1="27.94" x2="33.02" y2="25.4" width="0.1524" layer="91"/>
+<pinref part="GND15" gate="1" pin="GND"/>
+</segment>
+<segment>
+<pinref part="TP3" gate="G$1" pin="TP"/>
+<wire x1="63.5" y1="27.94" x2="73.66" y2="27.94" width="0.1524" layer="91"/>
+<wire x1="73.66" y1="27.94" x2="73.66" y2="25.4" width="0.1524" layer="91"/>
+<pinref part="GND16" gate="1" pin="GND"/>
+</segment>
 </net>
 <net name="+3V3" class="0">
@@
 <pinref part="R11" gate="G$1" pin="1"/>
 </segment>
+<segment>
+<pinref part="R3" gate="G$1" pin="1"/>
+<pinref part="+3V2" gate="G$1" pin="+3V3"/>
+<wire x1="73.66" y1="45.72" x2="73.66" y2="48.26" width="0.1524" layer="91"/>
+</segment>
 </net>
 <net name="S0" class="0">
@@
 <pinref part="P1" gate="G$1" pin="8"/>
 </segment>
+<segment>
+<pinref part="R1" gate="G$1" pin="2"/>
+<wire x1="40.64" y1="30.48" x2="48.26" y2="30.48" width="0.1524" layer="91"/>
+<wire x1="48.26" y1="30.48" x2="48.26" y2="35.56" width="0.1524" layer="91"/>
+<pinref part="P+15" gate="1" pin="+5V"/>
+</segment>
 </net>
 <net name="NEOPIXEL-SIGNAL" class="0">
@@
 </segment>
 </net>
+<net name="N$12" class="0">
+<segment>
+<pinref part="TP2" gate="G$1" pin="TP"/>
+<wire x1="22.86" y1="30.48" x2="30.48" y2="30.48" width="0.1524" layer="91"/>
+<pinref part="R1" gate="G$1" pin="1"/>
+</segment>
+</net>
