File: PCB/Root41-2020/002.brd (EAGLE design)
At the start: 72.1 x 74.3 mm, 37 parts, among them T1 NJL7502L, T10 NJL7502L, T11 NJL7502L, T2 NJL7502L, T3 NJL7502L, T4 NJL7502L, T5 NJL7502L, T6 NJL7502L, T7 NJL7502L, T8 NJL7502L, T9 NJL7502L

Commit message: ラインセンサできた
Parts:
- moved U$2 0.36 mm to (97.0, 7.00)
Changed lines of the file:
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@@
 <attribute name="VALUE" x="72.667" y="-3.81" size="0.4064" layer="27" rot="R90"/>
 </element>
-<element name="U$2" library="oshw" package="OSHW_5MM" value="" x="97.2" y="7.3" smashed="yes"/>
+<element name="U$2" library="oshw" package="OSHW_5MM" value="" x="97" y="7" smashed="yes"/>
 </elements>
 <signals>
@@
 <mfgpreviewcolor name="substratecolor" color="0xFF786E46"/>
 </mfgpreviewcolors>
+<errors>
+</errors>
 </board>
 </drawing>

Commit message: 基板設計完了
Other:
- board text added: "JLCJLCJLCJLC"
Changed lines of the file:
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@@
 <wire x1="91.83545" y1="-4.5" x2="49.24683125" y2="-4.5" width="0.01" layer="20"/>
 <wire x1="49.24683125" y1="-4.5" x2="48.74938125" y2="-4.949490625" width="0.01" layer="20" curve="84.2"/>
+<text x="43" y="-6" size="1.27" layer="21" font="vector" rot="R90">JLCJLCJLCJLC</text>
 </plain>
 <attributes>
@@
 </signals>
 <mfgpreviewcolors>
-<mfgpreviewcolor name="soldermaskcolor" color="0xC8008000"/>
+<mfgpreviewcolor name="soldermaskcolor" color="0xC8000000"/>
 <mfgpreviewcolor name="silkscreencolor" color="0xFFFEFEFE"/>
 <mfgpreviewcolor name="backgroundcolor" color="0xFF282828"/>
-<mfgpreviewcolor name="coppercolor" color="0xFFFFBF00"/>
+<mfgpreviewcolor name="coppercolor" color="0xFFECECEC"/>
 <mfgpreviewcolor name="substratecolor" color="0xFF786E46"/>
 </mfgpreviewcolors>
