File: PCB/Root41-2020/003.brd (EAGLE design)
At the start: 72.1 x 74.3 mm, 36 parts, among them T1 NJL7502L, T10 NJL7502L, T11 NJL7502L, T2 NJL7502L, T3 NJL7502L, T4 NJL7502L, T5 NJL7502L, T6 NJL7502L, T7 NJL7502L, T8 NJL7502L, T9 NJL7502L

Commit message: ラインセンサできた
Parts:
- added U$2: (no value), oshw:OSHW_5MM
- moved R15 0.70 mm to (-44.0, 10.3)
- moved R11 0.61 mm to (-41.9, -10.4), turned to 0 degrees
- turned T1 to 180 degrees
- turned T10 to 288 degrees
- turned T11 to 306 degrees
- turned T2 to 170.6 degrees
- turned T3 to 163.6 degrees
- turned T7 to 234 degrees
- turned T8 to 252 degrees
- turned T9 to 270 degrees
Routing:
- net S0: track 32.8 -> 75.0 mm, vias 2 -> 4
- net +5V: track 189.7 -> 157.2 mm, vias 2 -> 3
- net N$8: track 118.2 -> 102.2 mm, vias 0 -> 2
- net IN8: track 41.7 -> 25.6 mm, vias 4 -> 1
- net IN6: track 83.3 -> 69.3 mm
- net IN0: track 21.4 -> 33.8 mm, vias 0 -> 3
- net NEOPIXEL-SIGNAL: track 16.9 -> 25.9 mm, vias 1 -> 3
- net IN7: track 45.3 -> 54.2 mm
- net N$3: track 21.1 -> 28.7 mm
- net IN10: track 61.1 -> 53.6 mm, vias 0 -> 2
- net IN2: track 42.5 -> 49.3 mm
- net IN9: track 37.3 -> 44.0 mm, vias 1 -> 2
- net N$4: track 16.7 -> 22.2 mm
- net N$9: track 20.1 -> 24.3 mm
- net GND: track 209.6 -> 213.8 mm, vias 5 -> 4
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
Commit message: 基板設計完了
Other:
- board text added: "JLCJLCJLCJLC"
Changed lines of the file:
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@@
 <wire x1="-48.74938125" y1="-4.949490625" x2="-38.55565" y2="-30.24006875" width="0.01" layer="20" curve="32.310557"/>
 <wire x1="-38.635390625" y1="-31.56431875" x2="-38.55565" y2="-30.24006875" width="0.01" layer="20" curve="83.10798"/>
+<text x="-42" y="-6" size="1.27" layer="21" font="vector" rot="R90">JLCJLCJLCJLC</text>
 </plain>
 <attributes>
@@
 <element name="T3" library="#001-line" package="MYPARTS_NJL7502L" value="NJL7502L" x="-93.521" y="-27.571" smashed="yes" rot="MR163.6"/>
 <element name="T4" library="#001-line" package="MYPARTS_NJL7502L" value="NJL7502L" x="-85.083" y="0" smashed="yes" rot="MR180"/>
-<element name="T5" library="#001-line" package="MYPARTS_NJL7502L" value="NJL7502L" x="-72.667" y="0" smashed="yes" rot="MR180">
-<attribute name="NAME" x="-70.762" y="-0.381" size="1.27" layer="26" ratio="10" rot="MR180"/>
-</element>
+<element name="T5" library="#001-line" package="MYPARTS_NJL7502L" value="NJL7502L" x="-72.667" y="0" smashed="yes" rot="MR180"/>
 <element name="T6" library="#001-line" package="MYPARTS_NJL7502L" value="NJL7502L" x="-60.25" y="0" smashed="yes" rot="MR180"/>
 <element name="T7" library="#001-line" package="MYPARTS_NJL7502L" value="NJL7502L" x="-35.947" y="-26.117" smashed="yes" rot="MR234"/>
@@
 </signals>
 <mfgpreviewcolors>
-<mfgpreviewcolor name="soldermaskcolor" color="0xC8008000"/>
+<mfgpreviewcolor name="soldermaskcolor" color="0xC8000000"/>
 <mfgpreviewcolor name="silkscreencolor" color="0xFFFEFEFE"/>
 <mfgpreviewcolor name="backgroundcolor" color="0xFF282828"/>
-<mfgpreviewcolor name="coppercolor" color="0xFFFFBF00"/>
+<mfgpreviewcolor name="coppercolor" color="0xFFEDEDED"/>
 <mfgpreviewcolor name="substratecolor" color="0xFF786E46"/>
 </mfgpreviewcolors>
