File: PCB/Root41-2020/004.brd (EAGLE design)
At the start: 97 x 33.1 mm, 39 parts, among them T1 NJL7502L, T10 NJL7502L, T11 NJL7502L, T12 NJL7502L, T2 NJL7502L, T3 NJL7502L, T4 NJL7502L, T5 NJL7502L, T6 NJL7502L, T7 NJL7502L, T8 NJL7502L, T9 NJL7502L

Commit message: no message
Parts:
- removed R16: 120k, rcl:R0805
- added LED14: WS2812B5050, microbuilder:WS2812B
- added R1, R2: 120k, rcl:R0805
- added T13: NJL7502L, #001-line:MYPARTS_NJL7502L
- moved LED1 116.2 mm to (33.5, -91.6), turned to 339.9 degrees
- moved T1 110.7 mm to (27.9, -93.5)
- moved LED2 105.6 mm to (22.0, -95.0), turned to 346.9 degrees
- moved LED6 103.0 mm to (-33.5, -91.6), turned to 20.1 degrees
- moved R5 101.6 mm to (5.00, -99.0)
- moved T2 101.3 mm to (16.1, -96.2)
- moved T5 99.2 mm to (-27.9, -93.5)
- moved LED3 97.7 mm to (10.2, -97.0), turned to 354 degrees
- moved LED5 96.1 mm to (-22.0, -95.0), turned to 13.1 degrees
- moved R9 94.6 mm to (-6.00, -99.0)
- moved R6 94.6 mm to (5.00, -96.0)
- moved T3 94.4 mm to (0.00, -97.5)
- moved T4 93.1 mm to (-16.1, -96.2)
- moved LED7 92.6 mm to (0.00, -91.2), turned to 270 degrees
- moved LED4 92.5 mm to (-10.2, -97.0), turned to 6 degrees
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Connections:
- new net N$13: LED13.2-DOUT, LED14.4-DIN
- net +3V3: now also R1.1, R2.1; no longer R16.1
- net +5V: now also LED14.1-VDD
- net GND: now also LED14.3-GND, T13.E
- net IN11: now also R1.2; no longer R16.2
- net IN12: now also R2.2, T13.C
Routing:
- added copper zone on layer 1, net GND
- added copper zone on layer 16, net GND
Other:
- board size 97 x 33.1 mm -> 76.8 x 72.1 mm
- board text removed: "memo Y:-63mm"

Commit message: ラインセンサできた
Parts:
- added U$2: (no value), oshw:OSHW_5MM
- moved R13 4.24 mm to (17.0, -43.0), turned to 90 degrees
- turned T1 to 163.4 degrees
- turned T10 to 162 degrees
- turned T11 to 180 degrees
- flipped T12 to the bottom, turned to 198 degrees
- flipped T13 to the bottom, turned to 216 degrees
- turned T2 to 170.5 degrees
- turned T3 to 180 degrees
- turned T4 to 189.5 degrees
- turned T5 to 196.6 degrees
- turned T6 to 180 degrees
- turned T7 to 180 degrees
- turned T8 to 180 degrees
- turned T9 to 144 degrees
Routing:
- net GND: track 0.00 -> 293.3 mm, vias 0 -> 2
- net +5V: track 0.00 -> 207.1 mm, vias 0 -> 4
- net +3V3: track 0.00 -> 149.2 mm, vias 0 -> 5
- net NEOPIXEL-SIGNAL: track 0.00 -> 118.7 mm, vias 0 -> 3
- net IN4: track 0.00 -> 85.4 mm, vias 0 -> 3
- net IN8: track 0.00 -> 85.0 mm, vias 0 -> 2
- net IN0: track 0.00 -> 61.2 mm, vias 0 -> 2
- net IN3: track 0.00 -> 54.3 mm, vias 0 -> 3
- net IN2: track 0.00 -> 51.1 mm, vias 0 -> 3
- net IN1: track 0.00 -> 47.9 mm
- net N$6: track 0.00 -> 43.8 mm
- net N$10: track 0.00 -> 42.5 mm
- net IN12: track 0.00 -> 38.6 mm, vias 0 -> 2
- net IN9: track 0.00 -> 35.2 mm
- net S1: track 0.00 -> 28.9 mm, vias 0 -> 4
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
Commit message: 基板設計完了
Other:
- board text added: "JLCJLCJLCJLC"
Changed lines of the file:
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@@
 <circle x="-33.87868125" y="-38.12131875" radius="1.1" width="0.01" layer="20"/>
 <circle x="-33.159959375" y="-84.743240625" radius="1.1" width="0.01" layer="20"/>
+<text x="-5.2" y="-43" size="1.27" layer="21" font="vector">JLCJLCJLCJLC</text>
 </plain>
 <attributes>
@@
 <element name="LED2" library="microbuilder" package="WS2812B" value="WS2812B5050" x="22.019" y="-94.981" smashed="yes" rot="MR346.9"/>
 <element name="LED3" library="microbuilder" package="WS2812B" value="WS2812B5050" x="10.192" y="-96.966" smashed="yes" rot="MR354"/>
-<element name="LED4" library="microbuilder" package="WS2812B" value="WS2812B5050" x="-10.192" y="-96.966" smashed="yes" rot="MR6">
-<attribute name="NAME" x="-13.499425" y="-95.022128125" size="0.8128" layer="26" ratio="10" rot="MR276"/>
-</element>
-<element name="LED5" library="microbuilder" package="WS2812B" value="WS2812B5050" x="-22.019" y="-94.981" smashed="yes" rot="MR13.1">
-<attribute name="NAME" x="-25.0608" y="-92.64323125" size="0.8128" layer="26" ratio="10" rot="MR283.1"/>
-</element>
-<element name="LED6" library="microbuilder" package="WS2812B" value="WS2812B5050" x="-33.513" y="-91.56" smashed="yes" rot="MR20.1">
-<attribute name="NAME" x="-36.247225" y="-88.86895625" size="0.8128" layer="26" ratio="10" rot="MR290.1"/>
-</element>
+<element name="LED4" library="microbuilder" package="WS2812B" value="WS2812B5050" x="-10.192" y="-96.966" smashed="yes" rot="MR6"/>
+<element name="LED5" library="microbuilder" package="WS2812B" value="WS2812B5050" x="-22.019" y="-94.981" smashed="yes" rot="MR13.1"/>
+<element name="LED6" library="microbuilder" package="WS2812B" value="WS2812B5050" x="-33.513" y="-91.56" smashed="yes" rot="MR20.1"/>
 <element name="LED7" library="microbuilder" package="WS2812B" value="WS2812B5050" x="0" y="-91.214" smashed="yes" rot="MR270"/>
 <element name="LED8" library="microbuilder" package="WS2812B" value="WS2812B5050" x="0" y="-78.463" smashed="yes" rot="MR270"/>
-<element name="LED9" library="microbuilder" package="WS2812B" value="WS2812B5050" x="0" y="-66.071" smashed="yes" rot="MR270">
-<attribute name="NAME" x="-1.5875" y="-69.5635" size="0.8128" layer="26" ratio="10" rot="MR180"/>
-</element>
+<element name="LED9" library="microbuilder" package="WS2812B" value="WS2812B5050" x="0" y="-66.071" smashed="yes" rot="MR270"/>
 <element name="P1" library="zh" package="ZH-SM4-SIDE09" value="" x="8.863" y="-41.24" smashed="yes"/>
 <element name="R10" library="rcl" library_urn="urn:adsk.eagle:library:334" package="R0805" package3d_urn="urn:adsk.eagle:package:23553/2" value="120k" x="0" y="-82" smashed="yes">
@@
 <element name="T2" library="#001-line" package="MYPARTS_NJL7502L" value="NJL7502L" x="16.095" y="-96.18" smashed="yes" rot="MR170.5"/>
 <element name="T3" library="#001-line" package="MYPARTS_NJL7502L" value="NJL7502L" x="0" y="-97.5" smashed="yes" rot="MR180"/>
-<element name="T4" library="#001-line" package="MYPARTS_NJL7502L" value="NJL7502L" x="-16.095" y="-96.18" smashed="yes" rot="MR189.5">
-<attribute name="NAME" x="-14.27900625" y="-96.8701875" size="1.27" layer="26" ratio="10" rot="MR189.5"/>
-<attribute name="VALUE" x="-13.94363125" y="-94.86605625" size="1.27" layer="28" ratio="10" rot="MR189.5"/>
-</element>
-<element name="T5" library="#001-line" package="MYPARTS_NJL7502L" value="NJL7502L" x="-27.85" y="-93.478" smashed="yes" rot="MR196.6">
-<attribute name="NAME" x="-26.1332375" y="-94.387353125" size="1.27" layer="26" ratio="10" rot="MR196.6"/>
-<attribute name="VALUE" x="-25.552721875" y="-92.44004375" size="1.27" layer="28" ratio="10" rot="MR196.6"/>
-</element>
+<element name="T4" library="#001-line" package="MYPARTS_NJL7502L" value="NJL7502L" x="-16.095" y="-96.18" smashed="yes" rot="MR189.5"/>
+<element name="T5" library="#001-line" package="MYPARTS_NJL7502L" value="NJL7502L" x="-27.85" y="-93.478" smashed="yes" rot="MR196.6"/>
 <element name="T6" library="#001-line" package="MYPARTS_NJL7502L" value="NJL7502L" x="-0.18" y="-85" smashed="yes" rot="MR180"/>
 <element name="T7" library="#001-line" package="MYPARTS_NJL7502L" value="NJL7502L" x="0" y="-72.375" smashed="yes" rot="MR180"/>
@@
 </signals>
 <mfgpreviewcolors>
-<mfgpreviewcolor name="soldermaskcolor" color="0xC8008000"/>
+<mfgpreviewcolor name="soldermaskcolor" color="0xC8000000"/>
 <mfgpreviewcolor name="silkscreencolor" color="0xFFFEFEFE"/>
 <mfgpreviewcolor name="backgroundcolor" color="0xFF282828"/>
-<mfgpreviewcolor name="coppercolor" color="0xFFFFBF00"/>
+<mfgpreviewcolor name="coppercolor" color="0xFFF0F0F0"/>
 <mfgpreviewcolor name="substratecolor" color="0xFF786E46"/>
 </mfgpreviewcolors>
