File: PCB/Root41-2020/006.brd (EAGLE design)
At the start: 160 x 100 mm, 78 parts, among them IC1 MEGA8-AI, IC2 MEGA8-AI, P1 S6B-ZR-SM4A-TF, U1 IR2302STRPBF, U2 IR2302STRPBF, U3 IR2302STRPBF, U4 ATTINY85-20S, U5 IR2302STRPBF, U6 IR2302STRPBF, U7 IR2302STRPBF, X1 B2PS-VH, X2 B3PS-VH, X3 S3B-PH-SM4-TB, X5 B3PS-VH, X6 S3B-PH-SM4-TB, Y1 16Mhz, Y2 16Mhz

Commit message: 部品配置中
Parts:
- removed JP2: (no value), pinhead:2X03
- removed R28: 33k, rcl:R0603
- removed X5: B3PS-VH, con-JST VH:B3PS-VH
- removed X6: S3B-PH-SM4-TB, con-JST PH:S3B-PH-SM4-TB
- added CN1: (no value), jst-ph:B2B-PH-K-S
- added CN2, CN3: (no value), jst-ph:B3B-PH-K-S
- added R27: 33k, rcl:R0603
- JP1: device pinhead:2X03 -> pinhead:2X04
- X1: value B2PS-VH -> B2P-VH; device con-JST VH:B2PS-VH -> con-JST VH:B2P-VH
- X2: value B3PS-VH -> B3P-VH; device con-JST VH:B3PS-VH -> con-JST VH:B3P-VH
- X3: value S3B-PH-SM4-TB -> B3P-VH; device con-JST PH:S3B-PH-SM4-TB -> con-JST VH:B3P-VH
- moved Y2 93.3 mm to (-91.6, -4.38), flipped to the bottom, turned to 180 degrees
- moved R5 88.0 mm to (-78.5, -9.00), flipped to the bottom, turned to 180 degrees
- moved Y1 87.8 mm to (-89.2, -9.49), turned to 45 degrees
- moved R3 83.4 mm to (-82.4, 6.49), flipped to the bottom, turned to 180 degrees
- moved R7 78.9 mm to (-76.0, -2.50), flipped to the bottom
- moved C2 78.7 mm to (-88.4, -6.00), flipped to the bottom, turned to 270 degrees
- moved R17 77.8 mm to (-58.5, -6.00), flipped to the bottom
- moved C3 77.6 mm to (-78.5, -7.00), flipped to the bottom, turned to 180 degrees
- moved C8 75.9 mm to (-63.0, -12.0), flipped to the bottom, turned to 90 degrees
- moved R18 75.5 mm to (-58.5, -7.58), flipped to the bottom, turned to 180 degrees
- moved R11 75.2 mm to (-69.5, -2.50), flipped to the bottom, turned to 180 degrees
- moved C11 75.0 mm to (-90.0, -17.9), flipped to the bottom, turned to 90 degrees
- moved R20 74.6 mm to (-76.5, -10.5), flipped to the bottom, turned to 180 degrees
- moved R9 73.7 mm to (-66.0, -6.50), flipped to the bottom, turned to 270 degrees
- moved C7 72.5 mm to (-100.0, -0.50), turned to 180 degrees
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Connections:
- net !RESET2: now also JP1.7, R27.2; no longer JP2.5, R28.2
- net +5V: now also CN1.1, CN2.1, CN3.1, R27.1; no longer JP2.2, R28.1, X3.1, X6.1
- net ENC-1: now also CN2.3; no longer X3.2
- net ENC-2: now also CN3.3; no longer X6.2
- net GND: now also CN1.2, CN2.2, CN3.2; no longer JP2.6, X3.3, X6.3
- net MISO: no longer JP2.1
- net MOSI: no longer JP2.4
- net SCK: no longer JP2.3
- net U_BLDC-2CH: now also X3.1; no longer X5.1
- net V_BLDC-2CH: now also X3.2; no longer X5.2
- net W_BLDC-2CH: now also X3.3; no longer X5.3
Routing:
- net GND: track 0.00 -> 288.9 mm, vias 0 -> 42
- net VDD: track 0.00 -> 77.8 mm
- net W_BLDC-2CH: track 0.00 -> 49.4 mm
- net U_BLDC-1CH: track 0.00 -> 45.4 mm
- net V_BLDC-2CH: track 0.00 -> 30.1 mm
- net V_BLDC-1CH: track 0.00 -> 27.4 mm
- net U_BLDC-2CH: track 0.00 -> 27.1 mm
- net W_BLDC-1CH: track 0.00 -> 25.9 mm
- net N$25: track 0.00 -> 2.97 mm
- net N$20: track 0.00 -> 2.42 mm
- net N$26: track 0.00 -> 2.20 mm
- net N$21: track 0.00 -> 2.15 mm
Other:
- board size 160 x 100 mm -> 54.9 x 65.2 mm

Commit message: 配置完了！
Parts:
- moved R20 10.8 mm to (-72.5, -20.5), turned to 0 degrees
- moved R19 8.51 mm to (-76.0, -20.5)
- moved Y1 8.18 mm to (-97.0, -11.8), turned to 315 degrees
- moved R14 6.04 mm to (-95.0, 8.50), flipped to the top, turned to 270 degrees
- moved Y2 4.03 mm to (-91.1, -8.38)
- moved IC2 4.03 mm to (-94.3, -14.4)
- moved C2 3.95 mm to (-84.5, -6.60), turned to 0 degrees
- moved U2 3.00 mm to (-84.0, -3.00)
- moved R2 2.92 mm to (-82.5, 0.50), turned to 180 degrees
- moved IC1 1.80 mm to (-94.5, -5.50), turned to 45 degrees
- moved C3 1.50 mm to (-78.5, -5.50)
- moved D1 1.50 mm to (-77.5, -3.50)
- moved R5 1.50 mm to (-78.5, -7.50)
- moved R6 1.50 mm to (-76.0, -6.50)
- moved R7 1.50 mm to (-76.0, -1.00)
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Routing:
- net GND: track 288.9 -> 294.2 mm

Commit message: もうどうにでもなれ
Parts:
- added U$1: (no value), oshw:OSHW_5MM
- moved Q8 1.00 mm to (-68.0, -21.5)
Routing:
- net GND: track 294.2 -> 508.2 mm, vias 42 -> 49
- net +5V: track 0.00 -> 209.9 mm, vias 0 -> 7
- net MISO: track 0.00 -> 173.5 mm, vias 0 -> 14
- net EMERGENCY_R2: track 0.00 -> 167.0 mm, vias 0 -> 6
- net VDD: track 78.1 -> 218.3 mm, vias 0 -> 12
- net EMERGENCY_R1: track 0.00 -> 121.7 mm, vias 0 -> 6
- net EMERGENCY_T2: track 0.00 -> 105.5 mm, vias 0 -> 8
- net RX: track 0.00 -> 103.6 mm, vias 0 -> 6
- net ENC-2: track 0.00 -> 87.6 mm, vias 0 -> 4
- net V_IN-1CH: track 0.00 -> 83.5 mm, vias 0 -> 3
- net ENC-1: track 0.00 -> 69.6 mm, vias 0 -> 3
- net EMERGENCY_T1: track 0.00 -> 66.8 mm, vias 0 -> 3
- net N$37: track 0.00 -> 56.7 mm, vias 0 -> 2
- net N$14: track 0.00 -> 46.4 mm, vias 0 -> 1
- net MOSI: track 0.00 -> 39.8 mm, vias 0 -> 3
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- added copper zone on layer 1, net GND
- added copper zone on layer 16, net GND

Commit message: 基板設計完了
Connections:
- removed net SCK\: IC1.17, IC2.17
- net SCK: now also IC1.17, IC2.17
Routing:
- net SCK: track 0.00 -> 37.1 mm, vias 0 -> 11
- net SCK\: track 16.6 -> 0.00 mm, vias 3 -> 0
- net GND: track 508.2 -> 516.3 mm
- net EMERGENCY_T1: track 66.8 -> 68.3 mm
- net EMERGENCY_R2: track 167.0 -> 167.9 mm
- net EMERGENCY_R1: track 121.7 -> 122.2 mm
