File: PCB/Root41-2020/006.sch (EAGLE design)
At the start: 78 parts, among them IC1 MEGA8-AI, IC2 MEGA8-AI, P1 S6B-ZR-SM4A-TF, U1 IR2302STRPBF, U2 IR2302STRPBF, U3 IR2302STRPBF, U4 ATTINY85-20S, U5 IR2302STRPBF, U6 IR2302STRPBF, U7 IR2302STRPBF, X1 B2PS-VH, X2 B3PS-VH, X3 S3B-PH-SM4-TB, X5 B3PS-VH, X6 S3B-PH-SM4-TB, Y1 16Mhz, Y2 16Mhz

Commit message: 部品配置中
Parts:
- removed JP2: (no value), pinhead:PINHD-2X3
- removed R28: 33k, rcl:R-EU_R0603
- removed X5: B3PS-VH, con-JST VH:B3PS-VH
- removed X6: S3B-PH-SM4-TB, con-JST PH:S3B-PH-SM4-TB
- added CN1: (no value), jst-ph:B2B-PH-K-S
- added CN2, CN3: (no value), jst-ph:B3B-PH-K-S
- added R27: 33k, rcl:R-EU_R0603
- JP1: device pinhead:PINHD-2X3 -> pinhead:PINHD-2X4
- X1: value B2PS-VH -> B2P-VH; device con-JST VH:B2PS-VH -> con-JST VH:B2P-VH
- X2: value B3PS-VH -> B3P-VH; device con-JST VH:B3PS-VH -> con-JST VH:B3P-VH
- X3: value S3B-PH-SM4-TB -> B3P-VH; device con-JST PH:S3B-PH-SM4-TB -> con-JST VH:B3P-VH
Connections:
- net !RESET2: now also JP1.7, R27.2; no longer JP2.5, R28.2
- net +5V: now also CN1.1, CN2.1, CN3.1, R27.1; no longer JP2.2, R28.1, X3.1, X6.1
- net ENC-1: now also CN2.3; no longer X3.2
- net ENC-2: now also CN3.3; no longer X6.2
- net GND: now also CN1.2, CN2.2, CN3.2; no longer JP2.6, X3.3, X6.3
- net MISO: no longer JP2.1
- net MOSI: no longer JP2.4
- net SCK: no longer JP2.3
- net U_BLDC-2CH: now also X3.1; no longer X5.1
- net V_BLDC-2CH: now also X3.2; no longer X5.2
- net W_BLDC-2CH: now also X3.3; no longer X5.3

Commit message: 基板設計完了
Connections:
- removed net SCK\: IC1.PB5(SCK), IC2.PB5(SCK)
- net SCK: now also IC1.PB5(SCK), IC2.PB5(SCK)
Changed lines of the file:
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@@
-</segment>
-</net>
-<net name="SCK\" class="0">
-<segment>
-<pinref part="IC1" gate="G$1" pin="PB5(SCK)"/>
-<wire x1="86.36" y1="15.24" x2="101.6" y2="15.24" width="0.1524" layer="91"/>
-<label x="88.9" y="15.24" size="1.778" layer="95"/>
 </segment>
 </net>
@@
 <pinref part="JP1" gate="A" pin="3"/>
 </segment>
+<segment>
+<pinref part="IC1" gate="G$1" pin="PB5(SCK)"/>
+<wire x1="86.36" y1="15.24" x2="101.6" y2="15.24" width="0.1524" layer="91"/>
+<label x="88.9" y="15.24" size="1.778" layer="95"/>
+</segment>
 </net>
 <net name="EMERGENCY_T1" class="0">
@@
 </segment>
 </net>
-<net name="SCK\" class="0">
+<net name="SCK" class="0">
 <segment>
 <pinref part="IC2" gate="G$1" pin="PB5(SCK)"/>
