File: PCB/Root41-2020/007.brd (EAGLE design)
At the start: 54.9 x 65.2 mm, 79 parts, among them IC1 MEGA8-AI, IC2 MEGA8-AI, P1 S6B-ZR-SM4A-TF, U1 IR2302STRPBF, U2 IR2302STRPBF, U3 IR2302STRPBF, U4 ATTINY85-20S, U5 IR2302STRPBF, U6 IR2302STRPBF, U7 IR2302STRPBF, X1 B2P-VH, X2 B3P-VH, X3 B3P-VH, Y1 16Mhz, Y2 16Mhz

Commit message: 基板設計完了
Connections:
- removed net SCK\: IC1.17, IC2.17
- net SCK: now also IC1.17, IC2.17
Routing:
- net SCK: track 0.00 -> 43.4 mm, vias 0 -> 5
- net SCK\: track 36.5 -> 0.00 mm, vias 5 -> 0
- net N$14: track 28.4 -> 30.3 mm
