File: PCB/Root41-2020/007.sch (EAGLE design)
At the start: 78 parts, among them IC1 MEGA8-AI, IC2 MEGA8-AI, P1 S6B-ZR-SM4A-TF, U1 IR2302STRPBF, U2 IR2302STRPBF, U3 IR2302STRPBF, U4 ATTINY85-20S, U5 IR2302STRPBF, U6 IR2302STRPBF, U7 IR2302STRPBF, X1 B2P-VH, X2 B3P-VH, X3 B3P-VH, Y1 16Mhz, Y2 16Mhz

Commit message: 基板設計完了
Connections:
- removed net SCK\: IC1.PB5(SCK), IC2.PB5(SCK)
- net SCK: now also IC1.PB5(SCK), IC2.PB5(SCK)
Changed lines of the file:
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@@
 <setting verticaltext="up"/>
 </settings>
-<grid distance="0.1" unitdist="inch" unit="inch" style="lines" multiple="1" display="no" altdistance="0.01" altunitdist="inch" altunit="inch"/>
+<grid distance="0.1" unitdist="inch" unit="inch" style="lines" multiple="1" display="yes" altdistance="0.01" altunitdist="inch" altunit="inch"/>
 <layers>
 <layer number="1" name="Top" color="4" fill="1" visible="no" active="no"/>
@@
 </segment>
 </net>
-<net name="SCK\" class="0">
-<segment>
-<pinref part="IC1" gate="G$1" pin="PB5(SCK)"/>
-<wire x1="86.36" y1="15.24" x2="101.6" y2="15.24" width="0.1524" layer="91"/>
-<label x="88.9" y="15.24" size="1.778" layer="95"/>
-</segment>
-</net>
 <net name="MISO" class="0">
 <segment>
@@
 <pinref part="JP1" gate="A" pin="3"/>
 </segment>
+<segment>
+<pinref part="IC1" gate="G$1" pin="PB5(SCK)"/>
+<wire x1="86.36" y1="15.24" x2="101.6" y2="15.24" width="0.1524" layer="91"/>
+<label x="88.9" y="15.24" size="1.778" layer="95"/>
+</segment>
 </net>
 <net name="EMERGENCY_T1" class="0">
@@
 </segment>
 </net>
-<net name="SCK\" class="0">
+<net name="SCK" class="0">
 <segment>
 <pinref part="IC2" gate="G$1" pin="PB5(SCK)"/>
