File: PCB/Root41-2020/008.brd (EAGLE design)
At the start: 100 x 100 mm, 62 parts, among them IC1 MEGA8-AI, P1 S6B-ZR-SM4A-TF, Q1 BSS84

Commit message: 基板設計完了
Parts:
- added SJ1: (no value), jumper:SJ_2
- added TP18: TPSQTP10R, testpad:TP10R
- moved Q1 22.9 mm to (17.8, 27.9), turned to 270 degrees
- moved R4 17.3 mm to (14.0, 25.4), turned to 180 degrees
- moved TP1 0.64 mm to (8.26, -36.2)
- moved TP2 0.64 mm to (6.99, -36.2)
- moved TP4 0.64 mm to (4.45, -36.2)
- moved TP9 0.64 mm to (-3.17, -36.2)
- moved TP10 0.64 mm to (0.64, -36.2)
- moved TP11 0.64 mm to (-0.64, -36.2)
- moved TP6 0.64 mm to (1.91, -36.2)
- moved TP8 0.64 mm to (-1.91, -36.2)
- moved TP16 0.63 mm to (-6.99, -36.2)
- moved TP17 0.63 mm to (-5.71, -36.2)
- moved TP3 0.63 mm to (5.71, -36.2)
- moved TP5 0.63 mm to (3.17, -36.2)
- moved TP7 0.63 mm to (-4.45, -36.2)
Connections:
- new net CAM-UTIL: SJ1.2, SV1.13
- new net SWO: SV1.17, TP18.TP
- net RX-CAM: now also SJ1.3; no longer SV1.17
- net SS-CAM: now also SJ1.1; no longer SV1.13
Routing:
- net +5V: track 297.3 -> 441.7 mm, vias 2 -> 7
- net RX-CAM: track 85.0 -> 15.0 mm
- net CAM-UTIL: track 0.00 -> 64.7 mm, vias 0 -> 3
- net SS-CAM: track 66.3 -> 13.2 mm, vias 3 -> 0
- net RX-PC: track 37.9 -> 9.44 mm, vias 1 -> 0
- net BALL09: track 112.0 -> 87.9 mm
- net BALL_VIN: track 358.7 -> 340.0 mm
- net BALL14: track 56.0 -> 73.9 mm, vias 3 -> 1
- net GND: track 634.4 -> 619.0 mm, vias 53 -> 87
- net SCK: track 106.2 -> 121.1 mm, vias 3 -> 2
- net BALL16: track 26.7 -> 41.1 mm, vias 3 -> 2
- net NEOPIXEL: track 96.7 -> 110.2 mm
- net BALL06: track 60.1 -> 72.0 mm
- net BALL15: track 58.0 -> 46.8 mm
- net SS1: track 108.7 -> 98.0 mm, vias 1 -> 3
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Other:
- board text added: "JLCJLCJLCJLC"
