File: PCB/Root41-2020/008.sch (EAGLE design)
At the start: 61 parts, among them IC1 MEGA8-AI, P1 S6B-ZR-SM4A-TF, Q1 BSS84

Commit message: 基板設計完了
Parts:
- added SJ1: (no value), jumper:SJ2W
- added TP18: TPSQTP10R, testpad:TPSQTP10R
Connections:
- new net CAM-UTIL: SJ1.2, SV1.13
- new net SWO: SV1.17, TP18.TP
- net RX-CAM: now also SJ1.3; no longer SV1.17
- net SS-CAM: now also SJ1.1; no longer SV1.13
