File: PCB/Root41-2020/009.brd (EAGLE design)
At the start: 70 x 50 mm, 21 parts, among them U1 ATTINY85-20S

Commit message: 基板設計完了
Parts:
- added JP4: (no value), pinhead:1X08
- moved JP1 3.00 mm to (25.0, -14.0)
- moved U$1 2.00 mm to (-26.0, -9.00)
Connections:
- removed net RESET: TP5.TP
- new net SWO: JP1.10, JP3.14
- net !RESET: now also TP5.TP
- net +3V3: now also JP4.1
- net GND: now also JP4.2
- net SCL: now also JP4.3
- net SDA: now also JP4.4
Routing:
- net GND: track 159.8 -> 347.2 mm, vias 46 -> 35
- net SWO: track 0.00 -> 67.2 mm, vias 0 -> 2
- net +5V: track 40.5 -> 81.6 mm, vias 0 -> 1
- net +3V3: track 92.9 -> 133.2 mm, vias 2 -> 4
- net SW4: track 113.8 -> 81.3 mm, vias 3 -> 1
- net !RESET: track 0.00 -> 13.7 mm, vias 0 -> 1
- net TX-PC: track 42.7 -> 51.9 mm
- net SCL: track 67.0 -> 75.4 mm, vias 1 -> 0
- net UI: track 35.2 -> 43.2 mm, vias 1 -> 0
- net SW2: track 61.6 -> 56.8 mm
- net D+: track 31.7 -> 36.5 mm, vias 1 -> 0
- net RX-PC: track 39.0 -> 34.3 mm, vias 0 -> 1
- net SDA: track 71.2 -> 67.2 mm, vias 4 -> 1
- net SWDIO: track 23.0 -> 26.2 mm
- net SWCLK: track 19.1 -> 22.2 mm
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Other:
- board text added: "JLCJLCJLCJLC"
