File: PCB/Root41-2020/009.sch (EAGLE design)
At the start: 20 parts, among them U1 ATTINY85-20S

Commit message: 基板設計完了
Parts:
- added JP4: (no value), pinhead:PINHD-1X8
Connections:
- removed net RESET: TP5.TP
- new net SWO: JP1.10, JP3.14
- net !RESET: now also TP5.TP
- net +3V3: now also JP4.1
- net GND: now also JP4.2
- net SCL: now also JP4.3
- net SDA: now also JP4.4
Other:
- moved on the sheet: C1, CN1, JP1, JP2, R1, R2, R3, R4, S1, S2, S3, S4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
