File: PCB/Root41-2020/010.brd (EAGLE design)
At the start: 98 x 70 mm, 127 parts, among them Q2 TJ8S06M3L, Q3 IRLU3410PBF, U1 STM32F446RET6, U2 STMICROELECTRONICS_STM32L010F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, U3 STMICROELECTRONICS_STM32L010F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, U4 STMICROELECTRONICS_STM32L010F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, U5 STMICROELECTRONICS_STM32L010F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, X1 B4P-VH, X2 B3B-PH-K-S

Commit message: てめぇなんかにフィオをやれるか！
Parts:
- moved R5 10.8 mm to (-35.3, 5.33), turned to 0 degrees
- moved R6 9.90 mm to (-35.5, 1.22), turned to 90 degrees
- moved U4 2.00 mm to (-12.0, 35.0), turned to 90 degrees
- moved Q3 1.94 mm to (-11.0, 18.0)
- moved OK1 1.31 mm to (-42.5, 0.13)
- turned U5 to 270 degrees
Routing:
- net N$17: track 27.7 -> 31.4 mm
- net N$16: track 74.9 -> 75.7 mm
- net GND: track 165.3 -> 166.0 mm

Commit message: no message
Parts:
- removed Q3: IRLU3410PBF, myParts2:TO251AA
- added Q1: TO-252-NCH, Q:D-PAK_TO252AA
Connections:
- net GND: now also Q1.3; no longer Q3.3
- net N$17: now also Q1.4; no longer Q3.2, Q3.4
- net N$18: now also Q1.1; no longer Q3.1
Routing:
- net N$17: track 31.4 -> 23.8 mm
Changed lines of the file:
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@@
 <attribute name="VALUE" x="-31.259" y="17.852" size="1.27" layer="27" rot="R180"/>
-</element>
-<element name="Q3" library="myParts2" package="TO251AA" value="IRLU3410PBF" x="-10.984" y="18.039" smashed="yes">
-<attribute name="NAME" x="-13.524" y="21.849" size="1.27" layer="25"/>
-<attribute name="VALUE" x="-13.524" y="19.309" size="1.27" layer="27"/>
 </element>
 <element name="S1" library="switch-omron" library_urn="urn:adsk.eagle:library:377" package="B3F-10XX" package3d_urn="urn:adsk.eagle:package:27496/1" value="" x="-19" y="22" smashed="yes" rot="MR270">
@@
 <attribute name="VALUE" x="8.7899" y="15.24" size="0.02" layer="27"/>
 </element>
+<element name="Q1" library="Q" package="D-PAK_TO252AA" value="TO-252-NCH" x="-10" y="19" smashed="yes" rot="R45">
+<attribute name="NAME" x="-10.898025" y="14.509871875" size="1.27" layer="25" rot="R135"/>
+<attribute name="VALUE" x="-4.61184375" y="20.79605" size="1.27" layer="27" rot="R135"/>
+</element>
 </elements>
 <signals>
@@
 </signal>
 <signal name="N$17">
-<contactref element="Q3" pad="2"/>
-<contactref element="Q3" pad="4"/>
 <contactref element="CN1" pad="2"/>
-<wire x1="-10.984" y1="22.484" x2="-10.984" y2="23.53728125" width="3" layer="1"/>
 <wire x1="-25.5" y1="23.75" x2="-25.5" y2="26.5" width="1" layer="1"/>
-<wire x1="-24.5724" y1="27.4276" x2="-14.2926" y2="27.4276" width="1" layer="1"/>
-<wire x1="-10.984" y1="24.119" x2="-14.2926" y2="27.4276" width="1" layer="1"/>
-<wire x1="-10.984" y1="24.119" x2="-10.984" y2="22.484" width="1" layer="1"/>
 <wire x1="-25.5" y1="26.5" x2="-24.5724" y2="27.4276" width="1" layer="1"/>
-<wire x1="-10.984" y1="12.705" x2="-10.984" y2="22.349" width="1" layer="1"/>
-<wire x1="-10.984" y1="22.484" x2="-10.984" y2="22.349" width="0" layer="19" extent="1-1"/>
+<wire x1="-24.5724" y1="27.4276" x2="-14.4276" y2="27.4276" width="1" layer="1"/>
+<wire x1="-13" y1="26" x2="-13" y2="21.942975" width="1" layer="1"/>
+<wire x1="-14.4276" y1="27.4276" x2="-13" y2="26" width="1" layer="1"/>
+<contactref element="Q1" pad="4"/>
+<wire x1="-11.767765625" y1="20.767765625" x2="-10" y2="21" width="1" layer="1"/>
+<wire x1="-11.767765625" y1="20.767765625" x2="-13" y2="21.942975" width="1" layer="1"/>
 </signal>
 <signal name="N$18">
-<contactref element="Q3" pad="1"/>
 <contactref element="R3" pad="2"/>
 <contactref element="R4" pad="1"/>
+<contactref element="Q1" pad="1"/>
 <wire x1="-31.33" y1="-5.08" x2="-33.44" y2="-5.08" width="0" layer="19" extent="1-1"/>
-<wire x1="-13.27" y1="12.705" x2="-31.33" y2="-5.08" width="0" layer="19" extent="1-1"/>
+<wire x1="-8.218090625" y1="13.99368125" x2="-31.33" y2="-5.08" width="0" layer="19" extent="1-1"/>
 </signal>
 <signal name="N$19">
@@
 <contactref element="C3" pad="P$1"/>
 <contactref element="C4" pad="P$1"/>
-<contactref element="Q3" pad="3"/>
 <contactref element="JP2" pad="1"/>
 <contactref element="JP4" pad="1"/>
@@
 <contactref element="U$2" pad="P$2"/>
 <contactref element="TP35" pad="TP"/>
-<wire x1="14.3066" y1="10.3066" x2="-8.525" y2="10.3066" width="1" layer="1"/>
-<wire x1="-8.525" y1="10.3066" x2="-12.4404375" y2="10.3066" width="1" layer="1"/>
-<wire x1="14.3066" y1="10.3066" x2="16.5" y2="12.5" width="1" layer="1"/>
+<wire x1="16.3066" y1="12.3066" x2="16.5" y2="12.5" width="1" layer="1"/>
 <wire x1="-25" y1="17.5" x2="-22.77406875" y2="17.5" width="1" layer="1"/>
 <wire x1="-20.5724" y1="16.5724" x2="-16.5" y2="12.5" width="1" layer="1"/>
@@
 <wire x1="-28" y1="-12.93" x2="-28" y2="-12" width="0.2032" layer="1"/>
 <via x="-28" y="-12" extent="1-16" drill="0.35"/>
-<wire x1="-12.4404375" y1="10.3066" x2="-15.3066" y2="10.3066" width="1.016" layer="1"/>
-<wire x1="-15.3066" y1="10.3066" x2="-16.5" y2="11.5" width="1.016" layer="1"/>
-<wire x1="-16.5" y1="11.5" x2="-16.5" y2="12.5" width="1.016" layer="1"/>
-<wire x1="-8.698" y1="12.705" x2="-8.698" y2="10.4796" width="1" layer="1"/>
-<wire x1="-8.698" y1="10.4796" x2="-8.525" y2="10.3066" width="1" layer="1"/>
+<wire x1="-10.4404375" y1="12.3066" x2="-16.5" y2="12.3066" width="1.016" layer="1"/>
+<wire x1="-16.5" y1="12.3066" x2="-16.5" y2="12.5" width="1.016" layer="1"/>
+<contactref element="Q1" pad="3"/>
+<wire x1="-10.4404375" y1="12.3066" x2="-5" y2="12.3066" width="1" layer="1"/>
+<wire x1="-5" y1="12.3066" x2="16.3066" y2="12.3066" width="1" layer="1"/>
+<wire x1="-4.99368125" y1="17.218090625" x2="-4.99368125" y2="12.31291875" width="1" layer="1"/>
+<wire x1="-4.99368125" y1="12.31291875" x2="-5" y2="12.3066" width="1" layer="1"/>
 <wire x1="22.825" y1="39.675" x2="26" y2="38.15" width="0" layer="19" extent="1-1"/>
 <wire x1="22.85" y1="35" x2="26" y2="38.15" width="0" layer="19" extent="1-1"/>
@@
 <wire x1="-6.3144625" y1="23.681728125" x2="0" y2="24.55" width="0" layer="19" extent="1-16"/>
 <wire x1="-7.398959375" y1="21.39895625" x2="-6.3144625" y2="23.681728125" width="0" layer="19" extent="16-16"/>
+<wire x1="-4.99368125" y1="17.218090625" x2="-7.398959375" y2="21.39895625" width="0" layer="19" extent="1-16"/>
+<wire x1="26.67" y1="1.27" x2="22.101" y2="-1.27" width="0" layer="19" extent="1-1"/>
+<wire x1="30.48" y1="-0.635" x2="26.67" y2="1.27" width="0" layer="19" extent="1-16"/>
 <wire x1="-8.89" y1="30.06" x2="-6.3144625" y2="23.681728125" width="0" layer="19" extent="1-16"/>
 <wire x1="-11.69" y1="30" x2="-8.89" y2="30.06" width="0" layer="19" extent="1-1"/>
 <wire x1="-5.60104375" y1="31.39895625" x2="-8.89" y2="30.06" width="0" layer="19" extent="1-16"/>
-<wire x1="-11.675" y1="37.825" x2="-5.60104375" y2="31.39895625" width="0" layer="19" extent="1-16"/>
 <wire x1="-1.71826875" y1="31.7144625" x2="-5.60104375" y2="31.39895625" width="0" layer="19" extent="16-16"/>
-<wire x1="-8.698" y1="12.705" x2="-7.398959375" y2="21.39895625" width="0" layer="19" extent="16-16"/>
-<wire x1="26.67" y1="1.27" x2="22.101" y2="-1.27" width="0" layer="19" extent="1-1"/>
-<wire x1="30.48" y1="-0.635" x2="26.67" y2="1.27" width="0" layer="19" extent="1-16"/>
-<wire x1="7.15" y1="40" x2="9.675" y2="32.175" width="0" layer="19" extent="1-1"/>
+<wire x1="-11.675" y1="37.825" x2="-11.69" y2="30" width="0" layer="19" extent="1-1"/>
 <wire x1="-12.85" y1="40" x2="-11.675" y2="37.825" width="0" layer="19" extent="1-1"/>
 <wire x1="-17.175" y1="39.675" x2="-12.85" y2="40" width="0" layer="19" extent="1-1"/>
@@
 <wire x1="44.902" y1="7.176" x2="40.072" y2="4.886" width="0" layer="19" extent="1-1"/>
 <wire x1="44.902" y1="10.986" x2="44.902" y2="7.176" width="0" layer="19" extent="1-1"/>
+<wire x1="7.15" y1="40" x2="9.675" y2="32.175" width="0" layer="19" extent="1-1"/>
 <wire x1="-1.27" y1="43.18" x2="7.15" y2="40" width="0" layer="19" extent="1-1"/>
 <wire x1="8.89" y1="0.27" x2="18.669" y2="0" width="0" layer="19" extent="1-1"/>

Commit message: ひとまず配線終わったのだ！疲れたのだ！あとは電源基板とエンコーダ基板だけなのだ！
Routing:
- net GND: track 166.4 -> 606.1 mm, vias 2 -> 31
- net +3V3: track 40.0 -> 367.3 mm, vias 0 -> 20
- net SCL: track 0.00 -> 171.3 mm, vias 0 -> 14
- net SDA: track 0.00 -> 157.1 mm, vias 0 -> 14
- net +5V: track 76.3 -> 226.9 mm, vias 1 -> 13
- net SS-CAM: track 0.00 -> 99.6 mm, vias 0 -> 9
- net RADIO-OUT1: track 0.00 -> 95.3 mm, vias 0 -> 5
- net +12V: track 22.1 -> 114.2 mm, vias 1 -> 7
- net RADIO-RX: track 0.00 -> 91.3 mm, vias 0 -> 7
- net SPK-RX: track 0.00 -> 89.7 mm, vias 0 -> 5
- net NEOPIXEL: track 0.00 -> 87.3 mm, vias 0 -> 5
- net RADIO-OUT2: track 0.00 -> 85.1 mm, vias 0 -> 9
- net SPK-TX: track 0.00 -> 84.9 mm, vias 0 -> 3
- net RADIO-TX: track 0.00 -> 82.6 mm, vias 0 -> 5
- net MUX-B: track 0.00 -> 82.0 mm, vias 0 -> 5
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
Commit message: 基板設計完了
Parts:
- removed IC1: (no value), v-reg:TO220S
- added IC2: (no value), v-reg:78XXS
- added U$3: (no value), oshw:OSHW_5MM
- moved C16 4.77 mm to (16.6, -3.51)
- moved C14 0.50 mm to (19.1, 4.81)
Connections:
- net +12V: now also IC2.IN; no longer IC1.3
- net +5V: now also IC2.OUT; no longer IC1.2
- net GND: now also IC2.GND; no longer IC1.1
Routing:
- net GND: track 606.1 -> 618.8 mm, vias 31 -> 30
- net RADIO-OUT1: track 95.3 -> 93.5 mm
- net N$17: track 23.8 -> 22.0 mm
- net +5V: track 226.9 -> 227.6 mm
Other:
- board text added: "JLCJLCJLCJLC"
