File: PCB/Root41-2020/010.sch (EAGLE design)
At the start: 127 parts, among them Q2 TJ8S06M3L, Q3 IRLU3410PBF, U1 STM32F446RET6, U2 STMICROELECTRONICS_STM32L010F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, U3 STMICROELECTRONICS_STM32L010F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, U4 STMICROELECTRONICS_STM32L010F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, U5 STMICROELECTRONICS_STM32L010F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, X1 B4P-VH, X2 B3B-PH-K-S

Commit message: no message
Parts:
- removed Q3: IRLU3410PBF, myParts2:IRLU3410PBF
- added Q1: TO-252-NCH, Q:TO-252-NCH
Connections:
- net GND: now also Q1.S; no longer Q3.S
- net N$17: now also Q1.D; no longer Q3.D
- net N$18: now also Q1.G; no longer Q3.G
Changed lines of the file:
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@@
 <parts>
 <part name="Q2" library="transistor-fet" library_urn="urn:adsk.eagle:library:396" deviceset="SPD30P06P" device="TO252" package3d_urn="urn:adsk.eagle:package:28537/2" value="TJ8S06M3L"/>
-<part name="Q3" library="myParts2" deviceset="IRLU3410PBF" device=""/>
 <part name="C3" library="myParts2" deviceset="C12.5" device="" value="1000μ"/>
 <part name="OK1" library="optocoupler" library_urn="urn:adsk.eagle:library:320" deviceset="PC827" device="" package3d_urn="urn:adsk.eagle:package:21941/1" value="TLP621"/>
@@
 <part name="+3V22" library="supply1" library_urn="urn:adsk.eagle:library:371" deviceset="+3V3" device=""/>
 <part name="SJ4" library="jumper" library_urn="urn:adsk.eagle:library:252" deviceset="SJ2W" device="" package3d_urn="urn:adsk.eagle:package:15474/1"/>
+<part name="Q1" library="Q" deviceset="TO-252-NCH" device=""/>
 </parts>
 <sheets>
@@
 <attribute name="NAME" x="152.4" y="119.38" size="1.778" layer="95"/>
 </instance>
-<instance part="Q3" gate="G$1" x="213.36" y="88.9" smashed="yes">
-<attribute name="VALUE" x="218.44" y="86.36" size="1.778" layer="96"/>
-<attribute name="NAME" x="218.44" y="88.9" size="1.778" layer="95"/>
-</instance>
 <instance part="C3" gate="G$1" x="170.18" y="101.6" smashed="yes">
 <attribute name="NAME" x="160.782" y="101.6" size="1.778" layer="95"/>
@@
 <attribute name="NAME" x="167.64" y="114.7826" size="1.778" layer="95"/>
 <attribute name="VALUE" x="167.64" y="111.9886" size="1.778" layer="96"/>
+</instance>
+<instance part="Q1" gate="G$1" x="213.36" y="88.9" smashed="yes">
+<attribute name="NAME" x="220.98" y="91.44" size="1.778" layer="95"/>
+<attribute name="VALUE" x="220.98" y="88.9" size="1.778" layer="96"/>
 </instance>
 </instances>
@@
 <net name="N$17" class="0">
 <segment>
-<pinref part="Q3" gate="G$1" pin="D"/>
 <wire x1="215.9" y1="93.98" x2="215.9" y2="101.6" width="1.016" layer="91"/>
 <wire x1="215.9" y1="101.6" x2="226.06" y2="101.6" width="1.016" layer="91"/>
 <pinref part="CN1" gate="G$1" pin="2"/>
+<pinref part="Q1" gate="G$1" pin="D"/>
 </segment>
 </net>
 <net name="N$18" class="0">
 <segment>
-<pinref part="Q3" gate="G$1" pin="G"/>
 <wire x1="205.74" y1="86.36" x2="210.82" y2="86.36" width="0.1524" layer="91"/>
 <pinref part="R3" gate="G$1" pin="2"/>
 <pinref part="R4" gate="G$1" pin="1"/>
 <junction x="205.74" y="86.36"/>
+<pinref part="Q1" gate="G$1" pin="G"/>
 </segment>
 </net>
@@
 <wire x1="175.26" y1="96.52" x2="175.26" y2="76.2" width="1.016" layer="91"/>
 <junction x="175.26" y="76.2"/>
-<pinref part="Q3" gate="G$1" pin="S"/>
 <wire x1="215.9" y1="83.82" x2="215.9" y2="76.2" width="1.016" layer="91"/>
 <junction x="215.9" y="76.2"/>
@@
 <pinref part="R3" gate="G$1" pin="1"/>
 <junction x="205.74" y="76.2"/>
-</segment>
-<segment>
+<pinref part="Q1" gate="G$1" pin="S"/>
+</segment>
+<segment>

Commit message: 基板設計完了
Parts:
- removed IC1: (no value), v-reg:LM138-TS
- added IC2: (no value), v-reg:78XXS
Connections:
- net +12V: now also IC2.IN; no longer IC1.IN
- net +5V: now also IC2.OUT; no longer IC1.OUT
- net GND: now also IC2.GND; no longer IC1.ADJ
Changed lines of the file:
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@@
 <part name="GND44" library="supply1" library_urn="urn:adsk.eagle:library:371" deviceset="GND" device=""/>
 <part name="P+20" library="supply1" library_urn="urn:adsk.eagle:library:371" deviceset="+5V" device=""/>
-<part name="IC1" library="v-reg" library_urn="urn:adsk.eagle:library:409" deviceset="LM138-TS" device="" package3d_urn="urn:adsk.eagle:package:30366/1"/>
 <part name="R17" library="rcl" library_urn="urn:adsk.eagle:library:334" deviceset="R-TRIMM" device="3296W" package3d_urn="urn:adsk.eagle:package:26033/1" value="20k"/>
 <part name="GND45" library="supply1" library_urn="urn:adsk.eagle:library:371" deviceset="GND" device=""/>
@@
 <part name="SJ4" library="jumper" library_urn="urn:adsk.eagle:library:252" deviceset="SJ2W" device="" package3d_urn="urn:adsk.eagle:package:15474/1"/>
 <part name="Q1" library="Q" deviceset="TO-252-NCH" device=""/>
+<part name="IC2" library="v-reg" library_urn="urn:adsk.eagle:library:409" deviceset="78XXS" device="" package3d_urn="urn:adsk.eagle:package:30342/1"/>
 </parts>
 <sheets>
@@
 <attribute name="VALUE" x="101.6" y="116.84" size="1.778" layer="96"/>
 </instance>
-<instance part="IC1" gate="G$1" x="27.94" y="35.56" smashed="yes">
-<attribute name="NAME" x="30.48" y="27.94" size="1.778" layer="95"/>
-<attribute name="VALUE" x="30.48" y="25.4" size="1.778" layer="96"/>
-</instance>
 <instance part="R17" gate="G$1" x="116.84" y="30.48" smashed="yes">
 <attribute name="NAME" x="119.38" y="27.94" size="1.778" layer="95"/>
@@
 <attribute name="NAME" x="96.52" y="83.439" size="1.778" layer="95" rot="R180"/>
 <attribute name="VALUE" x="96.52" y="85.725" size="1.778" layer="96" rot="R180"/>
+</instance>
+<instance part="IC2" gate="1" x="27.94" y="35.56" smashed="yes">
+<attribute name="NAME" x="30.48" y="27.94" size="1.778" layer="95"/>
+<attribute name="VALUE" x="30.48" y="25.4" size="1.778" layer="96"/>
 </instance>
 </instances>
@@
 <pinref part="GND35" gate="1" pin="GND"/>
 <wire x1="27.94" y1="25.4" x2="27.94" y2="27.94" width="0.1524" layer="91"/>
-<pinref part="IC1" gate="G$1" pin="ADJ"/>
+<pinref part="IC2" gate="1" pin="GND"/>
 </segment>
 <segment>
@@
 <junction x="40.64" y="35.56"/>
 <pinref part="C14" gate="G$1" pin="+"/>
-<pinref part="IC1" gate="G$1" pin="OUT"/>
+<pinref part="IC2" gate="1" pin="OUT"/>
 </segment>
 <segment>
@@
 <wire x1="15.24" y1="33.02" x2="15.24" y2="35.56" width="0.1524" layer="91"/>
 <junction x="15.24" y="35.56"/>
-<pinref part="IC1" gate="G$1" pin="IN"/>
-</segment>
-<segment>
+<pinref part="IC2" gate="1" pin="IN"/>
+</segment>
+<segment>
